Commit message: Add qualified cuRobo previews with upright approach and ready stage

File: surgical_arm_bringup/config/curobo/gen3_surgical.urdf (robot description, URDF)
Before this commit: robot gen3, 16 links, 15 joints
Links:
- link base_link: geometry collision mesh filename=package://kortex_description/arms/gen3/7dof/meshes/base_lin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; visual mesh filename=package://kortex_description/arms/gen3/7dof/meshes/base_lin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
- link bracelet_link: geometry collision mesh filename=package://kortex_description/arms/gen3/7dof/meshes/bracelet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; visual mesh filename=package://kortex_description/arms/gen3/7dof/meshes/bracelet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
- link forearm_link: geometry collision mesh filename=package://kortex_description/arms/gen3/7dof/meshes/forearm_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; visual mesh filename=package://kortex_description/arms/gen3/7dof/meshes/forearm_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
- link half_arm_1_link: geometry collision mesh filename=package://kortex_description/arms/gen3/7dof/meshes/half_arm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; visual mesh filename=package://kortex_description/arms/gen3/7dof/meshes/half_arm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
- link half_arm_2_link: geometry collision mesh filename=package://kortex_description/arms/gen3/7dof/meshes/half_arm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; visual mesh filename=package://kortex_description/arms/gen3/7dof/meshes/half_arm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
- link shoulder_link: geometry collision mesh filename=package://kortex_description/arms/gen3/7dof/meshes/shoulder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; visual mesh filename=package://kortex_description/arms/gen3/7dof/meshes/shoulder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
- link spherical_wrist_1_link: geometry collision mesh filename=package://kortex_description/arms/gen3/7dof/meshes/spherica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; visual mesh filename=package://kortex_description/arms/gen3/7dof/meshes/spherica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
- link spherical_wrist_2_link: geometry collision mesh filename=package://kortex_description/arms/gen3/7dof/meshes/spherica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; visual mesh filename=package://kortex_description/arms/gen3/7dof/meshes/spherica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
- link thesis_ee: geometry collision mesh filename=package://kortex_description/grippers/thesis_ee/meshes/Full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 scale=0.001 0.001 0.001; collision mesh filename=package://kortex_description/grippers/thesis_ee/meshes/elbo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 scale=0.001 0.001 0.001
Joints:
- joint assembly_tip_joint: origin xyz=-0.027 0.000 -0.414 rpy=0 0 0 -> xyz=0.108 -0.008 -0.411 rpy=0 0 0

File: surgical_arm_bringup/config/curobo/gen3_surgical_resolved.urdf (robot description, URDF)
Before this commit: robot gen3, 16 links, 15 joints
Links:
- link base_link: geometry collision mesh filename=/home/kamren/workspace/ros2_kortex_ws/src/ros2_kortex/korte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; visual mesh filename=/home/kamren/workspace/ros2_kortex_ws/src/ros2_kortex/korte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
- link bracelet_link: geometry collision mesh filename=/home/kamren/workspace/ros2_kortex_ws/src/ros2_kortex/korte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; visual mesh filename=/home/kamren/workspace/ros2_kortex_ws/src/ros2_kortex/korte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
- link forearm_link: geometry collision mesh filename=/home/kamren/workspace/ros2_kortex_ws/src/ros2_kortex/korte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; visual mesh filename=/home/kamren/workspace/ros2_kortex_ws/src/ros2_kortex/korte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
- link half_arm_1_link: geometry collision mesh filename=/home/kamren/workspace/ros2_kortex_ws/src/ros2_kortex/korte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; visual mesh filename=/home/kamren/workspace/ros2_kortex_ws/src/ros2_kortex/korte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
- link half_arm_2_link: geometry collision mesh filename=/home/kamren/workspace/ros2_kortex_ws/src/ros2_kortex/korte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; visual mesh filename=/home/kamren/workspace/ros2_kortex_ws/src/ros2_kortex/korte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
- link shoulder_link: geometry collision mesh filename=/home/kamren/workspace/ros2_kortex_ws/src/ros2_kortex/korte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; visual mesh filename=/home/kamren/workspace/ros2_kortex_ws/src/ros2_kortex/korte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
- link spherical_wrist_1_link: geometry collision mesh filename=/home/kamren/workspace/ros2_kortex_ws/src/ros2_kortex/korte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; visual mesh filename=/home/kamren/workspace/ros2_kortex_ws/src/ros2_kortex/korte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
- link spherical_wrist_2_link: geometry collision mesh filename=/home/kamren/workspace/ros2_kortex_ws/src/ros2_kortex/korte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; visual mesh filename=/home/kamren/workspace/ros2_kortex_ws/src/ros2_kortex/korte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
- link thesis_ee: geometry collision mesh filename=/home/kamren/workspace/ros2_kortex_ws/src/ros2_kortex/korte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 scale=0.001 0.001 0.001; collision mesh filename=/home/kamren/workspace/ros2_kortex_ws/src/ros2_kortex/korte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 scale=0.001 0.001 0.001
Joints:
- joint assembly_tip_joint: origin xyz=-0.027 0.000 -0.414 rpy=0 0 0 -> xyz=0.108 -0.008 -0.411 rpy=0 0 0
